File: pcb/richkbd.kicad_pcb (KiCad board)
At the start: 2 copper layers, 315.3 x 126.9 mm, 67 parts, among them J2 OLED, SW1 SW_PUSH, SW10 SW_PUSH, SW11 SW_PUSH, SW12 SW_PUSH, SW13 SW_PUSH, SW14 SW_PUSH, SW15 SW_PUSH, SW16 SW_PUSH, SW17 SW_PUSH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

Commit message: Start of board layout
Parts:
- removed D1, D10, D11, D12, D13, D14, D15, D16, D17, D18, D19, D2, D20, D21, D3, D4, D5, D6, D7, D8, D9: D, kbd:D3_SMD
- removed J2: OLED, kbd:OLED
- removed L1, L10, L11, L12, L13, L14, L15, L16, L17, L18, L19, L2, L20, L21, L3, L4, L5, L6, L7, L8, L9: SK6812MINI, kbd:SK6812MINI_rev
- removed R1, R2: R, kbd:R
- removed RSW1: SW_PUSH, kbd:ResetSW
- added J1: USB_C_Receptacle, Connector_USB:USB_C_Receptacle_Amphenol_12401548E4-2A_CircularHoles, F.Cu at (184.3, 108.3)
- added K0: key-diode-led, nashlib:key_diode_led, F.Cu at (50.3, -86.0)
- added K1: key-diode-led, nashlib:key_diode_led, F.Cu at (69.7, -77.6)
- added K10: key-diode-led, nashlib:key_diode_led, F.Cu at (43.6, -64.3)
- added K11: key-diode-led, nashlib:key_diode_led, F.Cu at (62.9, -58.0)
- added K12: key-diode-led, nashlib:key_diode_led, F.Cu at (80.9, -51.2)
- added K13: key-diode-led, nashlib:key_diode_led, F.Cu at (101.1, -43.0)
- added K14: key-diode-led, nashlib:key_diode_led, F.Cu at (121.2, -35.2)
- added K15: key-diode-led, nashlib:key_diode_led, F.Cu at (141.2, -28.2)
- added K2: key-diode-led, nashlib:key_diode_led, F.Cu at (88.9, -71.6)
- added K20: key-diode-led, nashlib:key_diode_led, F.Cu at (28.8, -2.87)
- added K21: key-diode-led, nashlib:key_diode_led, F.Cu at (46.2, 4.04)
- added K22: key-diode-led, nashlib:key_diode_led, F.Cu at (65.6, 11.1)
- added K23: key-diode-led, nashlib:key_diode_led, F.Cu at (84.9, 20.1)
- added K24: key-diode-led, nashlib:key_diode_led, F.Cu at (105.1, 28.3)
- added K25: key-diode-led, nashlib:key_diode_led, F.Cu at (124.8, 34.5)
- added K3: key-diode-led, nashlib:key_diode_led, F.Cu at (108.2, -64.3)
- added K30: key-diode-led, nashlib:key_diode_led, F.Cu at (146.9, 210.3)
- added K31: key-diode-led, nashlib:key_diode_led, F.Cu at (166.5, 209.7)
- added K32: key-diode-led, nashlib:key_diode_led, F.Cu at (189.0, 209.5)
- added K33: key-diode-led, nashlib:key_diode_led, F.Cu at (208.9, 209.1)
- added K34: key-diode-led, nashlib:key_diode_led, F.Cu at (227.9, 207.6)
- added K35: key-diode-led, nashlib:key_diode_led, F.Cu at (248.8, 208.7)
- added K4: key-diode-led, nashlib:key_diode_led, F.Cu at (128.1, -55.1)
- added K40: key-diode-led, nashlib:key_diode_led, F.Cu at (253.6, 16.0)
- added K41: key-diode-led, nashlib:key_diode_led, F.Cu at (272.7, 8.89)
- added K42: key-diode-led, nashlib:key_diode_led, F.Cu at (290.0, 1.62)
- added K43: key-diode-led, nashlib:key_diode_led, F.Cu at (308.9, -4.79)
- added K44: key-diode-led, nashlib:key_diode_led, F.Cu at (328.7, -13.5)
- added K45: key-diode-led, nashlib:key_diode_led, F.Cu at (348.1, -20.2)
- added K5: key-diode-led, nashlib:key_diode_led, F.Cu at (147.6, -47.5)
- added K50: key-diode-led, nashlib:key_diode_led, F.Cu at (261.6, 34.6)
- added K51: key-diode-led, nashlib:key_diode_led, F.Cu at (281.4, 27.4)
- added K52: key-diode-led, nashlib:key_diode_led, F.Cu at (299.0, 20.5)
- added K53: key-diode-led, nashlib:key_diode_led, F.Cu at (318.7, 13.1)
- added K54: key-diode-led, nashlib:key_diode_led, F.Cu at (336.9, 5.60)
- added K55: key-diode-led, nashlib:key_diode_led, F.Cu at (356.5, -1.09)
- added K60: key-diode-led, nashlib:key_diode_led, F.Cu at (268.6, 54.2)
- added K61: key-diode-led, nashlib:key_diode_led, F.Cu at (288.4, 47.7)
- added K62: key-diode-led, nashlib:key_diode_led, F.Cu at (305.6, 41.3)
- added K63: key-diode-led, nashlib:key_diode_led, F.Cu at (324.4, 33.1)
- added K64: key-diode-led, nashlib:key_diode_led, F.Cu at (343.5, 25.6)
- added K65: key-diode-led, nashlib:key_diode_led, F.Cu at (364.3, 18.4)
Routing:
- removed copper zone on B.Cu, net GND
- removed copper zone on F.Cu, net GND
Other:
- outline, holes or cut-outs redrawn
- board text removed: "Corne Chocolate v2.1 PCB designed by foostan"
- board text removed: "GND"
- board text removed: "LED"
- board text removed: "OLED"
- board text removed: "VCC"

Commit message: switches laid
Parts:
- removed SW1, SW10, SW11, SW12, SW13, SW14, SW15, SW16, SW17, SW18, SW19, SW2, SW20, SW21, SW3, SW4, SW5, SW7, SW8, SW9: SW_PUSH, Switch_Keyboard_Hotswap_Kailh:Choc_Hotswap
- removed SW6: SW_PUSH, kbd:Choc_Hotswap
- added J2: OLED, kbd:OLED, F.Cu at (135.5, 138.1)
- added R1: R, kbd:R, F.Cu at (148.7, 137.8)
- added R2: R, kbd:R, F.Cu at (147.8, 96.7)
- added RSW1: SW_PUSH, kbd:ResetSW, F.Cu at (139.3, 97.5)
- added U1: ProMicro, kbd:ProMicro_v2, F.Cu at (141.8, 152.1)
- added U2: RP2040_Stamp, RP2040_Stamp:RP2040_Stamp_SMD, F.Cu at (140.6, 116.5)
- moved K45 199.5 mm to (189.2, 100.3), turned to -159 degrees
- moved K44 175.0 mm to (182.4, 82.6), turned to -159 degrees
- moved K3 164.7 mm to (37.2, 84.3)
- moved K2 164.5 mm to (19.4, 77.6)
- moved K55 154.5 mm to (211.1, 51.2), turned to -159 degrees
- moved K43 150.4 mm to (175.6, 64.8), turned to -159 degrees
- moved K42 149.8 mm to (158.7, 73.8), turned to -159 degrees
- moved K4 148.0 mm to (44.0, 66.6)
- moved K1 144.1 mm to (26.3, 59.8)
- moved K12 140.1 mm to (56.6, 86.7)
- moved K13 136.7 mm to (75.2, 91.3)
- moved K5 136.6 mm to (50.8, 48.9)
- moved K41 135.3 mm to (165.5, 91.6), turned to -159 degrees
- moved K54 134.8 mm to (217.9, 69.0), turned to -159 degrees
- moved K0 129.3 mm to (33.1, 42.1)
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Other:
- board size 315.3 x 126.9 mm -> 265.9 x 135.3 mm
