File: bottom_plate/richkbd_bottom_plate.kicad_pcb (KiCad board)
At the start: 2 copper layers, 265.9 x 119 mm, 9 parts, among them SW2 KEY_SWITCH

Commit message: A good start at the documentation.
Changed lines of the file:
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@@
       (effects (font (size 1 1) (thickness 0.15)))
     )
-    (fp_line (start 7 -7) (end -7 -7) (layer "Edge.Cuts") (width 0.12))
-    (fp_line (start -7 7) (end 7 7) (layer "Edge.Cuts") (width 0.12))
-    (fp_line (start 7 7) (end 7 -7) (layer "Edge.Cuts") (width 0.12))
-    (fp_line (start -7 -7) (end -7 7) (layer "Edge.Cuts") (width 0.12))
-    (fp_line (start 9.525 -9.525) (end -9.525 -9.525) (layer "F.Fab") (width 0.15))
-    (fp_line (start -9.525 -9.525) (end -9.525 9.525) (layer "F.Fab") (width 0.15))
-    (fp_line (start 9.525 9.525) (end 9.525 -9.525) (layer "F.Fab") (width 0.15))
-    (fp_line (start -9.525 9.525) (end 9.525 9.525) (layer "F.Fab") (width 0.15))
+    (fp_line (start 10.16 -10.16) (end -10.16 -10.16) (layer "Edge.Cuts") (width 0.12))
+    (fp_line (start -10.16 10.16) (end 10.16 10.16) (layer "Edge.Cuts") (width 0.12))
+    (fp_line (start 10.16 10.16) (end 10.16 -10.16) (layer "Edge.Cuts") (width 0.12))
+    (fp_line (start -10.16 -10.16) (end -10.16 10.16) (layer "Edge.Cuts") (width 0.12))
   )
   (footprint "" (layer "F.Cu")
