File: top_plate/richkbd_top_plate.kicad_pcb (KiCad board)
At the start: 2 copper layers, 265.9 x 119 mm, 50 parts, among them K0 key-diode-led, K1 key-diode-led, K10 key-diode-led, K100 key-diode-led, K101 key-diode-led, K102 key-diode-led, K11 key-diode-led, K110 key-diode-led, K111 key-diode-led, K112 key-diode-led, K12 key-diode-led, K2 key-diode-led, K20 key-diode-led, K21 key-diode-led, K22 key-diode-led, K30 key-diode-led, K31 key-diode-led, K32 key-diode-led, K33 key-diode-led, K40 key-diode-led, K41 key-diode-led, K42 key-diode-led, K43 key-diode-led, K50 key-diode-led, K51 key-diode-led, K52 key-diode-led, K53 key-diode-led, K60 key-diode-led, K61 key-diode-led, K62 key-diode-led, K63 key-diode-led, K70 key-diode-led, K71 key-diode-led, K72 key-diode-led, K73 key-diode-led, K80 key-diode-led, K81 key-diode-led, K82 key-diode-led, K83 key-diode-led, K90 key-diode-led, K91 key-diode-led, K92 key-diode-led

Commit message: Put stamp on the bottom layer
Parts:
- removed K100, K101, K102, K110, K111, K112, K60, K61, K62, K63, K70, K71, K72, K73, K80, K81, K82, K83, K90, K91, K92: key-diode-led, nashlib:Kailh_Switch_Hole
- removed case hole1: , 
- removed case hole2: , 
- removed case hole3: , 
- removed case hole4: , 
- moved K20 48.9 mm to (118.7, 45.2)
- moved K30 48.9 mm to (137.3, 49.8)
- moved K33 48.9 mm to (124.7, 109.2)
- moved K41 48.9 mm to (147.4, 76.6)
- moved K42 48.9 mm to (140.6, 94.3)
- moved case hole5 48.9 mm to (142.0, 64.1)
- moved K21 48.9 mm to (111.9, 62.9)
- moved K0 48.9 mm to (81.5, 36.0)
- moved K1 48.9 mm to (74.7, 53.7)
- moved K10 48.9 mm to (99.3, 42.8)
- moved K12 48.9 mm to (85.7, 78.2)
- moved K2 48.9 mm to (67.9, 71.5)
- moved K22 48.9 mm to (105.1, 80.7)
- moved K31 48.9 mm to (130.5, 67.5)
- moved K32 48.9 mm to (123.7, 85.2)
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Other:
- board size 265.9 x 119 mm -> 125.8 x 119 mm

Commit message: A good start at the documentation.
Other:
- board text added: "richkbd 2.0"
Changed lines of the file:
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@@
   (gr_line (start 159.887965 70.150621) (end 158.131936 74.725228) (layer "F.Fab") (width 0.1))
   (gr_line (start 156.722691 71.559894) (end 161.297233 73.315896) (layer "F.Fab") (width 0.1))
+  (gr_text "richkbd 2.0" (at 99.68 92.07 -21) (layer "F.SilkS")
+    (effects (font (size 1 1) (thickness 0.15)) (justify mirror))
+  )
+  (gr_text "richkbd 2.0" (at 99.66 92.08 -21) (layer "F.SilkS")
+    (effects (font (size 1 1) (thickness 0.15)))
+  )
 )
